File: Hardware/attiny1614.kicad_pcb (KiCad board)
At the start: 2 copper layers, 20.3 x 30.5 mm, 13 parts, among them J1 USB_C_Receptacle_USB2.0_14P, J2 Conn_01x03, J3 Conn_01x07, J4 Conn_01x07, U1 ATtiny1614-SS, U2 AP2112K-3.3

Commit message: Add files via upload
Routing:
- net Net-(U2-EN): track 8.62 -> 12.4 mm
- net +3V3: track 31.1 -> 32.6 mm
